File: disrabution_controler/hardware/distrabution_controler.kicad_sch (KiCad schematic)
At the start: 0 parts

Commit message: more hardware work
Other:
- removed sheet CAN_BUS
Changed lines of the file:
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@@
 	(paper "A4")
-	(sheet
-		(at 87.63 27.94)
-		(size 20.32 26.67)
-		(exclude_from_sim no)
-		(in_bom yes)
-		(on_board yes)
-		(dnp no)
-		(fields_autoplaced yes)
-		(stroke
-			(width 0.1524)
-			(type solid)
-		)
-		(fill
-			(color 0 0 0 0.0000)
-		)
-		(property "Sheetname" "CAN_BUS"
-			(at 87.63 27.2284 0)
-			(effects
-				(font
-					(size 1.27 1.27)
-				)
-				(justify left bottom)
-			)
-		)
-		(property "Sheetfile" "CAN_BUS.kicad_sch"
-			(at 87.63 55.1946 0)
-			(effects
-				(font
-					(size 1.27 1.27)
-				)
-				(justify left top)
-			)
-		)
-		(instances
-			(project "distrabution_controler"
-				(path "/2800815a-f06a-4e36-93dc-fea3151edeb4"
-					(page "4")
-				)
-			)
-		)
-	)
 	(sheet
 		(at 59.69 31.75)
