File: disrabution_controler/hardware/POWER_SUPPLY.kicad_sch (KiCad schematic)
At the start: 17 parts, among them Q18 NMOS, Q19 NMOS, U4 AP62150WU

Commit message: more hardware work
Other:
- moved on the sheet: C16, C17, C18, L1, Q18, Q19, R79, R80, R81, R82, R83, TP19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

Commit message: MORE PCB WORK
Parts:
- C32: renamed from C16; footprint (none) -> Capacitor_SMD:C_0603_1608Metric; Digikey Part Number (none) -> 399-C0603C104M5RACTUCT-ND
- C33: renamed from C18; footprint (none) -> Capacitor_SMD:C_0603_1608Metric; Digikey Part Number (none) -> 1276-1038-1-ND
- C34: renamed from C17; footprint (none) -> Capacitor_SMD:C_0603_1608Metric; Digikey Part Number (none) -> 490-7611-1-ND
- L1: footprint (none) -> Resistor_SMD:R_0603_1608Metric; Digikey Part Number (none) -> 445-173052-1-ND
- Q2: renamed from Q19; footprint (none) -> Resistor_SMD:R_0603_1608Metric; Digikey Part Number (none) -> BSS127H6327XTSA2CT-ND
- Q3: renamed from Q18; footprint (none) -> Resistor_SMD:R_0603_1608Metric; Digikey Part Number (none) -> BSS127H6327XTSA2CT-ND
- R51: renamed from R82; footprint (none) -> Resistor_SMD:R_0603_1608Metric; Digikey Part Number (none) -> 541-5351-1-ND
- R52: renamed from R81; footprint (none) -> Resistor_SMD:R_0603_1608Metric; Digikey Part Number (none) -> 541-100KHCT-ND
- R53: renamed from R83; footprint (none) -> Resistor_SMD:R_0603_1608Metric; Digikey Part Number (none) -> RMCF0603JT10K0CT-ND
- R54: renamed from R80; footprint (none) -> Resistor_SMD:R_0603_1608Metric; Digikey Part Number (none) -> 541-100KHCT-ND
- R55: renamed from R79; footprint (none) -> Resistor_SMD:R_0603_1608Metric; Digikey Part Number (none) -> RMCF0603JT10K0CT-ND
- TP25: renamed from TP20; footprint (none) -> TestPoint:TestPoint_Pad_D1.0mm; now left out of the parts list
- TP26: renamed from TP19; footprint (none) -> TestPoint:TestPoint_Pad_D1.0mm; now left out of the parts list
- TP27: renamed from TP22; footprint (none) -> TestPoint:TestPoint_Pad_D1.0mm; now left out of the parts list
- TP28: renamed from TP21; footprint (none) -> TestPoint:TestPoint_Pad_D1.0mm; now left out of the parts list
- TP29: renamed from TP23; footprint (none) -> TestPoint:TestPoint_Pad_D1.0mm; now left out of the parts list
- U7: renamed from U4; Digikey Part Number (none) -> 31-AP62150WU-7CT-ND

Commit message: more hardware work on disrabution controler nearing ifc
Parts:
- added H20, H21, H22, H23, H24: MountingHole, MountingHole:MountingHole_4.3mm_M4, symbol Mechanical:MountingHole
- L1: footprint Resistor_SMD:R_0603_1608Metric -> L_Bourns_SDR0604
- Q2, Q3: footprint Resistor_SMD:R_0603_1608Metric -> Package_TO_SOT_SMD:SOT-23
Connections:
- net ALLOW_Q_DRAW: now also Q3.1 (G); no longer Q3.2 (G)
- net GND: now also Q2.2 (S), Q3.2 (S); no longer Q2.3 (S), Q3.3 (S)
- net at R52.1, TP27.1, U7.5 (EN): now also Q2.3 (D); no longer Q2.1 (D)
- net at R54.1, TP28.1: now also Q2.1 (G), Q3.3 (D); no longer Q2.2 (G), Q3.1 (D)
