File: disrabution_controler/hardware/DISTRABUTION.kicad_sch (KiCad schematic)
At the start: 116 parts, among them Q1 PMOS, Q10 PMOS, Q11 PMOS, Q12 PMOS, Q13 PMOS, Q14 PMOS, Q15 PMOS, Q16 PMOS, Q2 PMOS, Q3 PMOS, Q4 PMOS, Q5 PMOS, Q6 PMOS, Q7 PMOS, Q8 PMOS, Q9 PMOS

Commit message: more hardware work
Parts:
- added D18: SK6805, LED_SMD:LED_SK6805_PLCC4_2.4x2.7mm_P1.3mm, symbol LED:SK6805
- added F17: Fuse_Small, symbol Device:Fuse_Small
- added Q20: PMOS, symbol Simulation_SPICE:PMOS
- added R88: 10K, symbol Device:R
- added R89: R, symbol Device:R
- added TP31: ~, symbol Connector:TestPoint
Connections:
- net +12V: now also Q20.3 (S), R88.1
- net +3V3: now also D18.4 (VDD)
- net GND: now also D18.2 (VSS)
- net at D13.1 (DOUT): now also D18.3 (DIN)
- new net: Q20.1 (D), R89.1
- new net PERIPHERAL_PWR: F17.1
- new net PERIPHERAL_PWR_CSN: F17.2, R89.2
- new net PERIPHERAL_PWR_GATE: Q20.2 (G), R88.2, TP31.1
Other:
- moved on the sheet: D10, D11, D12, D13, D14, D15, D16, D17, D2, D3, D4, D5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

Commit message: MORE PCB WORK
Parts:
- removed Q20: PMOS, symbol Simulation_SPICE:PMOS
- added Q20: PMOS, Package_SO:Vishay_PowerPAK_1212-8_Single, symbol LIBRAY:SiSS27DN
- D1: renamed from D2; value SK6805 -> SK6805-EC; Digikey Part Number (none) -> 1528-4492-ND
- D10: renamed from D13; value SK6805 -> SK6805-EC; Digikey Part Number (none) -> 1528-4492-ND
- D11: renamed from D12; value SK6805 -> SK6805-EC; Digikey Part Number (none) -> 1528-4492-ND
- D12: renamed from D11; value SK6805 -> SK6805-EC; Digikey Part Number (none) -> 1528-4492-ND
- D13: renamed from D10; value SK6805 -> SK6805-EC; Digikey Part Number (none) -> 1528-4492-ND
- D14, D15, D16, D17: value SK6805 -> SK6805-EC; Digikey Part Number (none) -> 1528-4492-ND
- D2: renamed from D3; value SK6805 -> SK6805-EC; Digikey Part Number (none) -> 1528-4492-ND
- D3: renamed from D4; value SK6805 -> SK6805-EC; Digikey Part Number (none) -> 1528-4492-ND
- D4: renamed from D5; value SK6805 -> SK6805-EC; Digikey Part Number (none) -> 1528-4492-ND
- D5: renamed from D6; value SK6805 -> SK6805-EC; Digikey Part Number (none) -> 1528-4492-ND
- D6: renamed from D7; value SK6805 -> SK6805-EC; Digikey Part Number (none) -> 1528-4492-ND
- D7: renamed from D8; value SK6805 -> SK6805-EC; Digikey Part Number (none) -> 1528-4492-ND
- D8: renamed from D9; value SK6805 -> SK6805-EC; Digikey Part Number (none) -> 1528-4492-ND
- D9: renamed from D18; value SK6805 -> SK6805-EC; Digikey Part Number (none) -> 1528-4492-ND
- F1, F10, F11, F12, F13, F14, F15, F16, F17, F2, F3, F4, F5, F6, F7, F8, F9: footprint (none) -> Library:ATO_FUSEHOLDER; Digikey Part Number (none) -> 36-3522-ND
- H1, H10, H11, H12, H13, H14, H15, H16, H19, H2, H3, H4, H5, H6, H7, H8, H9: footprint (none) -> MountingHole:MountingHole_6.4mm_M6_Pad_TopOnly
- H17, H18: footprint (none) -> MountingHole:MountingHole_8.4mm_M8_Pad_TopOnly
- Q10: renamed from Q7; footprint (none) -> Package_SO:Vishay_PowerPAK_1212-8_Single; symbol Simulation_SPICE:PMOS -> LIBRAY:SiSS27DN
- Q11: renamed from Q8; footprint (none) -> Package_SO:Vishay_PowerPAK_1212-8_Single; symbol Simulation_SPICE:PMOS -> LIBRAY:SiSS27DN
- Q12: renamed from Q9; footprint (none) -> Package_SO:Vishay_PowerPAK_1212-8_Single; symbol Simulation_SPICE:PMOS -> LIBRAY:SiSS27DN
- Q13: renamed from Q10; footprint (none) -> Package_SO:Vishay_PowerPAK_1212-8_Single; symbol Simulation_SPICE:PMOS -> LIBRAY:SiSS27DN
- Q14: renamed from Q11; footprint (none) -> Package_SO:Vishay_PowerPAK_1212-8_Single; symbol Simulation_SPICE:PMOS -> LIBRAY:SiSS27DN
- Q15: renamed from Q12; footprint (none) -> Package_SO:Vishay_PowerPAK_1212-8_Single; symbol Simulation_SPICE:PMOS -> LIBRAY:SiSS27DN
- Q16: renamed from Q13; footprint (none) -> Package_SO:Vishay_PowerPAK_1212-8_Single; symbol Simulation_SPICE:PMOS -> LIBRAY:SiSS27DN
- Q17: renamed from Q14; footprint (none) -> Package_SO:Vishay_PowerPAK_1212-8_Single; symbol Simulation_SPICE:PMOS -> LIBRAY:SiSS27DN
- Q18: renamed from Q15; footprint (none) -> Package_SO:Vishay_PowerPAK_1212-8_Single; symbol Simulation_SPICE:PMOS -> LIBRAY:SiSS27DN
- Q19: renamed from Q16; footprint (none) -> Package_SO:Vishay_PowerPAK_1212-8_Single; symbol Simulation_SPICE:PMOS -> LIBRAY:SiSS27DN
- Q4: footprint (none) -> Package_SO:Vishay_PowerPAK_1212-8_Single; symbol Simulation_SPICE:PMOS -> LIBRAY:SiSS27DN
- Q5: renamed from Q1; footprint (none) -> Package_SO:Vishay_PowerPAK_1212-8_Single; symbol Simulation_SPICE:PMOS -> LIBRAY:SiSS27DN
- Q6: renamed from Q2; footprint (none) -> Package_SO:Vishay_PowerPAK_1212-8_Single; symbol Simulation_SPICE:PMOS -> LIBRAY:SiSS27DN
- Q7: renamed from Q3; footprint (none) -> Package_SO:Vishay_PowerPAK_1212-8_Single; symbol Simulation_SPICE:PMOS -> LIBRAY:SiSS27DN
- Q8: renamed from Q5; footprint (none) -> Package_SO:Vishay_PowerPAK_1212-8_Single; symbol Simulation_SPICE:PMOS -> LIBRAY:SiSS27DN
- Q9: renamed from Q6; footprint (none) -> Package_SO:Vishay_PowerPAK_1212-8_Single; symbol Simulation_SPICE:PMOS -> LIBRAY:SiSS27DN
- R56: renamed from R3; footprint (none) -> Resistor_SMD:R_0603_1608Metric; Digikey Part Number (none) -> RMCF0603JT10K0CT-ND
- R57: renamed from R6; footprint (none) -> Resistor_SMD:R_0603_1608Metric; Digikey Part Number (none) -> RMCF0603JT10K0CT-ND
- R58: renamed from R8; footprint (none) -> Resistor_SMD:R_0603_1608Metric; Digikey Part Number (none) -> RMCF0603JT10K0CT-ND
- R59: renamed from R10; footprint (none) -> Resistor_SMD:R_0603_1608Metric; Digikey Part Number (none) -> RMCF0603JT10K0CT-ND
- R60: renamed from R12; footprint (none) -> Resistor_SMD:R_0603_1608Metric; Digikey Part Number (none) -> RMCF0603JT10K0CT-ND
- R61: renamed from R14; footprint (none) -> Resistor_SMD:R_0603_1608Metric; Digikey Part Number (none) -> RMCF0603JT10K0CT-ND
- R62: renamed from R16; footprint (none) -> Resistor_SMD:R_0603_1608Metric; Digikey Part Number (none) -> RMCF0603JT10K0CT-ND
- R63: renamed from R18; footprint (none) -> Resistor_SMD:R_0603_1608Metric; Digikey Part Number (none) -> RMCF0603JT10K0CT-ND
- R64: renamed from R4; value R -> R002; footprint (none) -> Resistor_SMD:R_2512_6332Metric; Digikey Part Number (none) -> CRF2512-FZ-R002ELFCT-ND
- R65: renamed from R7; value R -> R002; footprint (none) -> Resistor_SMD:R_2512_6332Metric; Digikey Part Number (none) -> CRF2512-FZ-R002ELFCT-ND
- R66: renamed from R9; value R -> R002; footprint (none) -> Resistor_SMD:R_2512_6332Metric; Digikey Part Number (none) -> CRF2512-FZ-R002ELFCT-ND
- R67: renamed from R11; value R -> R002; footprint (none) -> Resistor_SMD:R_2512_6332Metric; Digikey Part Number (none) -> CRF2512-FZ-R002ELFCT-ND
- R68: renamed from R13; value R -> R002; footprint (none) -> Resistor_SMD:R_2512_6332Metric; Digikey Part Number (none) -> CRF2512-FZ-R002ELFCT-ND
- R69: renamed from R15; value R -> R002; footprint (none) -> Resistor_SMD:R_2512_6332Metric; Digikey Part Number (none) -> CRF2512-FZ-R002ELFCT-ND
- R70: renamed from R17; value R -> R002; footprint (none) -> Resistor_SMD:R_2512_6332Metric; Digikey Part Number (none) -> CRF2512-FZ-R002ELFCT-ND
- R71: renamed from R19; value R -> R002; footprint (none) -> Resistor_SMD:R_2512_6332Metric; Digikey Part Number (none) -> CRF2512-FZ-R002ELFCT-ND
- R72: renamed from R20; footprint (none) -> Resistor_SMD:R_0603_1608Metric; Digikey Part Number (none) -> RMCF0603JT10K0CT-ND
- R73: renamed from R22; footprint (none) -> Resistor_SMD:R_0603_1608Metric; Digikey Part Number (none) -> RMCF0603JT10K0CT-ND
- R74: renamed from R24; footprint (none) -> Resistor_SMD:R_0603_1608Metric; Digikey Part Number (none) -> RMCF0603JT10K0CT-ND
- R75: renamed from R26; footprint (none) -> Resistor_SMD:R_0603_1608Metric; Digikey Part Number (none) -> RMCF0603JT10K0CT-ND
- R76: renamed from R28; footprint (none) -> Resistor_SMD:R_0603_1608Metric; Digikey Part Number (none) -> RMCF0603JT10K0CT-ND
- R77: renamed from R30; footprint (none) -> Resistor_SMD:R_0603_1608Metric; Digikey Part Number (none) -> RMCF0603JT10K0CT-ND
- R78: renamed from R32; footprint (none) -> Resistor_SMD:R_0603_1608Metric; Digikey Part Number (none) -> RMCF0603JT10K0CT-ND
- R79: renamed from R34; footprint (none) -> Resistor_SMD:R_0603_1608Metric; Digikey Part Number (none) -> RMCF0603JT10K0CT-ND
- R80: renamed from R21; value R -> R002; footprint (none) -> Resistor_SMD:R_2512_6332Metric; Digikey Part Number (none) -> CRF2512-FZ-R002ELFCT-ND
- R81: renamed from R23; value R -> R002; footprint (none) -> Resistor_SMD:R_2512_6332Metric; Digikey Part Number (none) -> CRF2512-FZ-R002ELFCT-ND
- R82: renamed from R25; value R -> R002; footprint (none) -> Resistor_SMD:R_2512_6332Metric; Digikey Part Number (none) -> CRF2512-FZ-R002ELFCT-ND
- R83: renamed from R27; value R -> R002; footprint (none) -> Resistor_SMD:R_2512_6332Metric; Digikey Part Number (none) -> CRF2512-FZ-R002ELFCT-ND
- R84: renamed from R29; value R -> R002; footprint (none) -> Resistor_SMD:R_2512_6332Metric; Digikey Part Number (none) -> CRF2512-FZ-R002ELFCT-ND
- R85: renamed from R31; value R -> R002; footprint (none) -> Resistor_SMD:R_2512_6332Metric; Digikey Part Number (none) -> CRF2512-FZ-R002ELFCT-ND
- R86: renamed from R33; value R -> R002; footprint (none) -> Resistor_SMD:R_2512_6332Metric; Digikey Part Number (none) -> CRF2512-FZ-R002ELFCT-ND
- R87: renamed from R35; value R -> R002; footprint (none) -> Resistor_SMD:R_2512_6332Metric; Digikey Part Number (none) -> CRF2512-FZ-R002ELFCT-ND
- R88: footprint (none) -> Resistor_SMD:R_0603_1608Metric; Digikey Part Number (none) -> RMCF0603JT10K0CT-ND
- R89: value R -> R002; footprint (none) -> Resistor_SMD:R_2512_6332Metric; Digikey Part Number (none) -> CRF2512-FZ-R002ELFCT-ND
- TP30: renamed from TP1; footprint (none) -> TestPoint:TestPoint_Pad_D1.0mm; now left out of the parts list
- TP31: renamed from TP2; footprint (none) -> TestPoint:TestPoint_Pad_D1.0mm; now left out of the parts list
- TP32: renamed from TP3; footprint (none) -> TestPoint:TestPoint_Pad_D1.0mm; now left out of the parts list
- TP33: renamed from TP4; footprint (none) -> TestPoint:TestPoint_Pad_D1.0mm; now left out of the parts list
- TP34: renamed from TP5; footprint (none) -> TestPoint:TestPoint_Pad_D1.0mm; now left out of the parts list
- TP35: renamed from TP6; footprint (none) -> TestPoint:TestPoint_Pad_D1.0mm; now left out of the parts list
- TP36: renamed from TP7; footprint (none) -> TestPoint:TestPoint_Pad_D1.0mm; now left out of the parts list
- TP37: renamed from TP8; footprint (none) -> TestPoint:TestPoint_Pad_D1.0mm; now left out of the parts list
- TP38: renamed from TP9; footprint (none) -> TestPoint:TestPoint_Pad_D1.0mm; now left out of the parts list
- TP39: renamed from TP10; footprint (none) -> TestPoint:TestPoint_Pad_D1.0mm; now left out of the parts list
- TP40: renamed from TP11; footprint (none) -> TestPoint:TestPoint_Pad_D1.0mm; now left out of the parts list
- TP41: renamed from TP12; footprint (none) -> TestPoint:TestPoint_Pad_D1.0mm; now left out of the parts list
- TP42: renamed from TP13; footprint (none) -> TestPoint:TestPoint_Pad_D1.0mm; now left out of the parts list
- TP43: renamed from TP14; footprint (none) -> TestPoint:TestPoint_Pad_D1.0mm; now left out of the parts list
- TP44: renamed from TP16; footprint (none) -> TestPoint:TestPoint_Pad_D1.0mm; now left out of the parts list
- TP45: renamed from TP17; footprint (none) -> TestPoint:TestPoint_Pad_D1.0mm; now left out of the parts list
- TP46: renamed from TP18; footprint (none) -> TestPoint:TestPoint_Pad_D1.0mm; now left out of the parts list
- TP47: renamed from TP31; footprint (none) -> TestPoint:TestPoint_Pad_D1.0mm; now left out of the parts list
Connections:
- net +12V: now also Q10.1 (S), Q10.2 (S), Q11.1 (S), Q11.2 (S), Q12.1 (S), Q12.2 (S), Q13.1 (S), Q13.2 (S), Q14.1 (S), Q14.2 (S), Q15.1 (S), Q15.2 (S), Q16.1 (S), Q16.2 (S), Q17.1 (S), Q17.2 (S), Q18.1 (S), Q18.2 (S), Q19.1 (S), Q19.2 (S), Q4.1 (S), Q4.2 (S), Q5.1 (S), Q5.2 (S), Q6.1 (S), Q6.2 (S), Q7.1 (S), Q7.2 (S), Q8.1 (S), Q8.2 (S), Q9.1 (S), Q9.2 (S), Q20.1 (S), Q20.2 (S), Q20.3 (S)
- net CH10_GATE: now also Q13.4 (G); no longer Q13.2 (G)
- net CH11_GATE: now also Q14.4 (G); no longer Q14.2 (G)
- net CH12_GATE: now also Q15.4 (G); no longer Q15.2 (G)
- net CH13_GATE: now also Q16.4 (G); no longer Q16.2 (G)
- net CH14_GATE: now also Q17.4 (G); no longer Q17.2 (G)
- net CH15_GATE: now also Q18.4 (G); no longer Q18.2 (G)
- net CH16_GATE: now also Q19.4 (G); no longer Q19.2 (G)
- net CH1_GATE: now also Q4.4 (G); no longer Q4.2 (G)
- net CH2_GATE: now also Q5.4 (G); no longer Q5.2 (G)
- net CH3_GATE: now also Q6.4 (G); no longer Q6.2 (G)
- net CH4_GATE: now also Q7.4 (G); no longer Q7.2 (G)
- net CH5_GATE: now also Q8.4 (G); no longer Q8.2 (G)
- net CH6_GATE: now also Q9.4 (G); no longer Q9.2 (G)
- net CH7_GATE: now also Q10.4 (G); no longer Q10.2 (G)
- net CH8_GATE: now also Q11.4 (G); no longer Q11.2 (G)
- net CH9_GATE: now also Q12.4 (G); no longer Q12.2 (G)
- net PERIPHERAL_PWR_GATE: now also Q20.4 (G)
- net at R80.1: now also Q12.5 (D); no longer Q12.1 (D)
- net at R64.1: now also Q4.5 (D); no longer Q4.1 (D)
- net at R89.1: now also Q20.5 (D)
- net at R83.1: now also Q15.5 (D); no longer Q15.1 (D)
- net at R67.1: now also Q7.5 (D); no longer Q7.1 (D)
- net at R66.1: now also Q6.5 (D); no longer Q6.1 (D)
- net at R86.1: now also Q18.5 (D); no longer Q18.1 (D)
- net at R81.1: now also Q13.5 (D); no longer Q13.1 (D)
- net at R69.1: now also Q9.5 (D); no longer Q9.1 (D)
- net at R87.1: now also Q19.5 (D); no longer Q19.1 (D)
- net at R82.1: now also Q14.5 (D); no longer Q14.1 (D)
- net at R71.1: now also Q11.5 (D); no longer Q11.1 (D)
- net at R68.1: now also Q8.5 (D); no longer Q8.1 (D)
- net at R70.1: now also Q10.5 (D); no longer Q10.1 (D)
- net at R84.1: now also Q16.5 (D); no longer Q16.1 (D)
- net at R85.1: now also Q17.5 (D); no longer Q17.1 (D)
- net at R65.1: now also Q5.5 (D); no longer Q5.1 (D)

Commit message: working on firmware but notaced a hardware issue
Parts:
- added Q21, Q22, Q23, Q24, Q25, Q26, Q27, Q28, Q29, Q30, Q31, Q32, Q33, Q34, Q35, Q36, Q37: NMOS, Package_TO_SOT_SMD:SOT-23, symbol Simulation_SPICE:NMOS
- added TP48, TP49, TP50, TP51, TP52, TP53, TP54, TP55, TP56, TP57, TP58, TP59, TP60, TP61, TP62, TP63, TP64: ~, TestPoint:TestPoint_Pad_D1.0mm, symbol Connector:TestPoint
- F1, F10, F11, F12, F13, F14, F15, F16, F17, F2, F3, F4, F5, F6, F7, F8, F9: value Fuse_Small -> ~
Connections:
- net CH10_GATE: now also Q31.1 (G), TP57.1; no longer Q13.4 (G), R73.2, TP39.1
- net CH11_GATE: now also Q32.1 (G), TP58.1; no longer Q14.4 (G), R74.2, TP40.1
- net CH12_GATE: now also Q33.1 (G), TP59.1; no longer Q15.4 (G), R75.2, TP41.1
- net CH13_GATE: now also Q34.1 (G), TP60.1; no longer Q16.4 (G), R76.2, TP42.1
- net CH14_GATE: now also Q35.1 (G), TP61.1; no longer Q17.4 (G), R77.2, TP43.1
- net CH15_GATE: now also Q36.1 (G), TP62.1; no longer Q18.4 (G), R78.2, TP44.1
- net CH16_GATE: now also Q37.1 (G), TP63.1; no longer Q19.4 (G), R79.2, TP45.1
- net CH1_GATE: now also Q21.1 (G), TP48.1; no longer Q4.4 (G), R56.2, TP30.1
- net CH2_GATE: now also Q22.1 (G), TP49.1; no longer Q5.4 (G), R57.2, TP31.1
- net CH3_GATE: now also Q23.1 (G), TP50.1; no longer Q6.4 (G), R58.2, TP32.1
- net CH4_GATE: now also Q25.1 (G), TP51.1; no longer Q7.4 (G), R59.2, TP33.1
- net CH5_GATE: now also Q26.1 (G), TP52.1; no longer Q8.4 (G), R60.2, TP34.1
- net CH6_GATE: now also Q27.1 (G), TP53.1; no longer Q9.4 (G), R61.2, TP35.1
- net CH7_GATE: now also Q28.1 (G), TP54.1; no longer Q10.4 (G), R62.2, TP36.1
- net CH8_GATE: now also Q29.1 (G), TP55.1; no longer Q11.4 (G), R63.2, TP37.1
- net CH9_GATE: now also Q30.1 (G), TP56.1; no longer Q12.4 (G), R72.2, TP38.1
- net GND: now also Q21.2 (S), Q22.2 (S), Q23.2 (S), Q24.2 (S), Q25.2 (S), Q26.2 (S), Q27.2 (S), Q28.2 (S), Q29.2 (S), Q30.2 (S), Q31.2 (S), Q32.2 (S), Q33.2 (S), Q34.2 (S), Q35.2 (S), Q36.2 (S), Q37.2 (S)
- net PERIPHERAL_PWR_GATE: now also Q24.1 (G), TP64.1; no longer Q20.4 (G), R88.2, TP47.1
- new net: Q15.4 (G), Q33.3 (D), R75.2, TP41.1
- new net: Q21.3 (D), Q4.4 (G), R56.2, TP30.1
- new net: Q17.4 (G), Q35.3 (D), R77.2, TP43.1
- new net: Q14.4 (G), Q32.3 (D), R74.2, TP40.1
- new net: Q12.4 (G), Q30.3 (D), R72.2, TP38.1
- new net: Q19.4 (G), Q37.3 (D), R79.2, TP45.1
- new net: Q11.4 (G), Q29.3 (D), R63.2, TP37.1
- new net: Q18.4 (G), Q36.3 (D), R78.2, TP44.1
- new net: Q23.3 (D), Q6.4 (G), R58.2, TP32.1
- new net: Q25.3 (D), Q7.4 (G), R59.2, TP33.1
- new net: Q16.4 (G), Q34.3 (D), R76.2, TP42.1
- new net: Q22.3 (D), Q5.4 (G), R57.2, TP31.1
- new net: Q10.4 (G), Q28.3 (D), R62.2, TP36.1
- new net: Q27.3 (D), Q9.4 (G), R61.2, TP35.1
- new net: Q20.4 (G), Q24.3 (D), R88.2, TP47.1
- new net: Q13.4 (G), Q31.3 (D), R73.2, TP39.1
- new net: Q26.3 (D), Q8.4 (G), R60.2, TP34.1
Other:
- moved on the sheet: F1, F10, F11, F12, F13, F14, F15, F16, F2, F3, F4, F5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
