File: disrabution_controler/hardware/ANALOUGE.kicad_sch (KiCad schematic)
At the start: 66 parts, among them U1 ADS7128, U12 ADS7128

Commit message: MORE PCB WORK
Parts:
- C24: renamed from C50; value 0.1uF -> 0uF1; Digikey Part Number (none) -> 399-C0603C104M5RACTUCT-ND
- C25: renamed from C51; value 0.1uF -> 0uF1; Digikey Part Number (none) -> 399-C0603C104M5RACTUCT-ND
- C26: renamed from C52; Digikey Part Number (none) -> 1276-1038-1-ND
- C27: renamed from C49; Digikey Part Number (none) -> 1276-1946-1-ND
- C28: renamed from C2; value 0.1uF -> 0uF1; Digikey Part Number (none) -> 399-C0603C104M5RACTUCT-ND
- C29: renamed from C3; value 0.1uF -> 0uF1; Digikey Part Number (none) -> 399-C0603C104M5RACTUCT-ND
- C30: renamed from C4; Digikey Part Number (none) -> 1276-1038-1-ND
- C31: renamed from C1; Digikey Part Number (none) -> 1276-1946-1-ND
- R13: renamed from R36; footprint (none) -> Resistor_SMD:R_0603_1608Metric; Digikey Part Number (none) -> RMCF0603JT10K0CT-ND
- R14: renamed from R38; footprint (none) -> Resistor_SMD:R_0603_1608Metric; Digikey Part Number (none) -> RMCF0603JT10K0CT-ND
- R15: renamed from R40; footprint (none) -> Resistor_SMD:R_0603_1608Metric; Digikey Part Number (none) -> RMCF0603JT10K0CT-ND
- R16: renamed from R42; footprint (none) -> Resistor_SMD:R_0603_1608Metric; Digikey Part Number (none) -> RMCF0603JT10K0CT-ND
- R17: renamed from R44; footprint (none) -> Resistor_SMD:R_0603_1608Metric; Digikey Part Number (none) -> RMCF0603JT10K0CT-ND
- R18: renamed from R46; footprint (none) -> Resistor_SMD:R_0603_1608Metric; Digikey Part Number (none) -> RMCF0603JT10K0CT-ND
- R19: renamed from R48; footprint (none) -> Resistor_SMD:R_0603_1608Metric; Digikey Part Number (none) -> RMCF0603JT10K0CT-ND
- R20: renamed from R52; footprint (none) -> Resistor_SMD:R_0603_1608Metric; Digikey Part Number (none) -> RMCF0603JT10K0CT-ND
- R21: renamed from R86; footprint (none) -> Resistor_SMD:R_0603_1608Metric; Digikey Part Number (none) -> RMCF0603JT10K0CT-ND
- R22: renamed from R72; footprint (none) -> Resistor_SMD:R_0603_1608Metric; Digikey Part Number (none) -> RMCF0603JT10K0CT-ND
- R23: renamed from R62; Digikey Part Number (none) -> 541-0.0GCT-ND
- R24: renamed from R37; footprint (none) -> Resistor_SMD:R_0603_1608Metric; Digikey Part Number (none) -> 311-20.0KHRCT-ND
- R25: renamed from R39; footprint (none) -> Resistor_SMD:R_0603_1608Metric; Digikey Part Number (none) -> 311-20.0KHRCT-ND
- R26: renamed from R41; footprint (none) -> Resistor_SMD:R_0603_1608Metric; Digikey Part Number (none) -> 311-20.0KHRCT-ND
- R27: renamed from R43; footprint (none) -> Resistor_SMD:R_0603_1608Metric; Digikey Part Number (none) -> 311-20.0KHRCT-ND
- R28: renamed from R45; footprint (none) -> Resistor_SMD:R_0603_1608Metric; Digikey Part Number (none) -> 311-20.0KHRCT-ND
- R29: renamed from R47; footprint (none) -> Resistor_SMD:R_0603_1608Metric; Digikey Part Number (none) -> 311-20.0KHRCT-ND
- R30: renamed from R49; footprint (none) -> Resistor_SMD:R_0603_1608Metric; Digikey Part Number (none) -> 311-20.0KHRCT-ND
- R31: renamed from R53; footprint (none) -> Resistor_SMD:R_0603_1608Metric; Digikey Part Number (none) -> 311-20.0KHRCT-ND
- R32: renamed from R87; footprint (none) -> Resistor_SMD:R_0603_1608Metric; Digikey Part Number (none) -> 311-20.0KHRCT-ND
- R33: renamed from R73; footprint (none) -> Resistor_SMD:R_0603_1608Metric; Digikey Part Number (none) -> 311-20.0KHRCT-ND
- R34: renamed from R54; footprint (none) -> Resistor_SMD:R_0603_1608Metric; Digikey Part Number (none) -> RMCF0603JT10K0CT-ND
- R35: renamed from R56; footprint (none) -> Resistor_SMD:R_0603_1608Metric; Digikey Part Number (none) -> RMCF0603JT10K0CT-ND
- R36: renamed from R58; footprint (none) -> Resistor_SMD:R_0603_1608Metric; Digikey Part Number (none) -> RMCF0603JT10K0CT-ND
- R37: renamed from R61; footprint (none) -> Resistor_SMD:R_0603_1608Metric; Digikey Part Number (none) -> RMCF0603JT10K0CT-ND
- R38: renamed from R64; footprint (none) -> Resistor_SMD:R_0603_1608Metric; Digikey Part Number (none) -> RMCF0603JT10K0CT-ND
- R39: renamed from R66; footprint (none) -> Resistor_SMD:R_0603_1608Metric; Digikey Part Number (none) -> RMCF0603JT10K0CT-ND
- R40: renamed from R68; footprint (none) -> Resistor_SMD:R_0603_1608Metric; Digikey Part Number (none) -> RMCF0603JT10K0CT-ND
- R41: renamed from R70; footprint (none) -> Resistor_SMD:R_0603_1608Metric; Digikey Part Number (none) -> RMCF0603JT10K0CT-ND
- R42: renamed from R1; Digikey Part Number (none) -> 541-100KHCT-ND
- R43: renamed from R55; footprint (none) -> Resistor_SMD:R_0603_1608Metric; Digikey Part Number (none) -> 311-20.0KHRCT-ND
- R44: renamed from R57; footprint (none) -> Resistor_SMD:R_0603_1608Metric; Digikey Part Number (none) -> 311-20.0KHRCT-ND
- R45: renamed from R60; footprint (none) -> Resistor_SMD:R_0603_1608Metric; Digikey Part Number (none) -> 311-20.0KHRCT-ND
- R46: renamed from R63; footprint (none) -> Resistor_SMD:R_0603_1608Metric; Digikey Part Number (none) -> 311-20.0KHRCT-ND
- R47: renamed from R65; footprint (none) -> Resistor_SMD:R_0603_1608Metric; Digikey Part Number (none) -> 311-20.0KHRCT-ND
- R48: renamed from R67; footprint (none) -> Resistor_SMD:R_0603_1608Metric; Digikey Part Number (none) -> 311-20.0KHRCT-ND
- R49: renamed from R69; footprint (none) -> Resistor_SMD:R_0603_1608Metric; Digikey Part Number (none) -> 311-20.0KHRCT-ND
- R50: renamed from R71; footprint (none) -> Resistor_SMD:R_0603_1608Metric; Digikey Part Number (none) -> 311-20.0KHRCT-ND
- TP10: renamed from TP41; footprint (none) -> TestPoint:TestPoint_Pad_D1.0mm; now left out of the parts list
- TP11: renamed from TP42; footprint (none) -> TestPoint:TestPoint_Pad_D1.0mm; now left out of the parts list
- TP12: renamed from TP43; footprint (none) -> TestPoint:TestPoint_Pad_D1.0mm; now left out of the parts list
- TP13: renamed from TP44; footprint (none) -> TestPoint:TestPoint_Pad_D1.0mm; now left out of the parts list
- TP14: renamed from TP45; footprint (none) -> TestPoint:TestPoint_Pad_D1.0mm; now left out of the parts list
- TP15: renamed from TP46; footprint (none) -> TestPoint:TestPoint_Pad_D1.0mm; now left out of the parts list
- TP16: renamed from TP47; footprint (none) -> TestPoint:TestPoint_Pad_D1.0mm; now left out of the parts list
- TP17: renamed from TP32; footprint (none) -> TestPoint:TestPoint_Pad_D1.0mm; now left out of the parts list
- TP18: renamed from TP33; footprint (none) -> TestPoint:TestPoint_Pad_D1.0mm; now left out of the parts list
- TP19: renamed from TP34; footprint (none) -> TestPoint:TestPoint_Pad_D1.0mm; now left out of the parts list
- TP20: renamed from TP35; footprint (none) -> TestPoint:TestPoint_Pad_D1.0mm; now left out of the parts list
- TP21: renamed from TP36; footprint (none) -> TestPoint:TestPoint_Pad_D1.0mm; now left out of the parts list
- TP22: renamed from TP37; footprint (none) -> TestPoint:TestPoint_Pad_D1.0mm; now left out of the parts list
- TP23: renamed from TP38; footprint (none) -> TestPoint:TestPoint_Pad_D1.0mm; now left out of the parts list
- TP24: renamed from TP39; footprint (none) -> TestPoint:TestPoint_Pad_D1.0mm; now left out of the parts list
- TP7: renamed from TP30; footprint (none) -> TestPoint:TestPoint_Pad_D1.0mm; now left out of the parts list
- TP8: renamed from TP26; footprint (none) -> TestPoint:TestPoint_Pad_D1.0mm; now left out of the parts list
- TP9: renamed from TP40; footprint (none) -> TestPoint:TestPoint_Pad_D1.0mm; now left out of the parts list
- U5: renamed from U12; Digikey Part Number (none) -> 296-ADS7128IRTERCT-ND
- U6: renamed from U1; Digikey Part Number (none) -> 296-ADS7128IRTERCT-ND
Connections:
- net CH10_CSN_DEV: now also TP18.1, U6.5 (AIN6/GPIO6); no longer TP23.1, U6.16 (AIN1/GPIO1)
- net CH11_CSN_DEV: now also TP19.1, U6.4 (AIN5/GPIO5); no longer TP22.1, U6.1 (AIN2/GPIO2)
- net CH12_CSN_DEV: now also TP20.1, U6.3 (AIN4/GPIO4); no longer TP21.1, U6.2 (AIN3/GPIO3)
- net CH13_CSN_DEV: now also TP21.1, U6.2 (AIN3/GPIO3); no longer TP20.1, U6.3 (AIN4/GPIO4)
- net CH14_CSN_DEV: now also TP22.1, U6.1 (AIN2/GPIO2); no longer TP19.1, U6.4 (AIN5/GPIO5)
- net CH15_CSN_DEV: now also TP23.1, U6.16 (AIN1/GPIO1); no longer TP18.1, U6.5 (AIN6/GPIO6)
- net CH16_CSN_DEV: now also TP24.1, U6.15 (AIN0/GPIO0); no longer TP17.1, U6.6 (AIN7/GPIO7)
- net CH1_CSN_DEV: now also TP9.1, U5.6 (AIN7/GPIO7); no longer TP16.1, U5.15 (AIN0/GPIO0)
- net CH2_CSN_DEV: now also TP10.1, U5.5 (AIN6/GPIO6); no longer TP15.1, U5.16 (AIN1/GPIO1)
- net CH3_CSN_DEV: now also TP11.1, U5.4 (AIN5/GPIO5); no longer TP14.1, U5.1 (AIN2/GPIO2)
- net CH4_CSN_DEV: now also TP12.1, U5.3 (AIN4/GPIO4); no longer TP13.1, U5.2 (AIN3/GPIO3)
- net CH5_CSN_DEV: now also TP13.1, U5.2 (AIN3/GPIO3); no longer TP12.1, U5.3 (AIN4/GPIO4)
- net CH6_CSN_DEV: now also TP14.1, U5.1 (AIN2/GPIO2); no longer TP11.1, U5.4 (AIN5/GPIO5)
- net CH7_CSN_DEV: now also TP15.1, U5.16 (AIN1/GPIO1); no longer TP10.1, U5.5 (AIN6/GPIO6)
- net CH8_CSN_DEV: now also TP16.1, U5.15 (AIN0/GPIO0); no longer TP9.1, U5.6 (AIN7/GPIO7)
- net CH9_CSN_DEV: now also TP17.1, U6.6 (AIN7/GPIO7); no longer TP24.1, U6.15 (AIN0/GPIO0)
- net ADC_ALERT renamed ADC_01_ALERT
- net ADC_01_ALERT: no longer U6.12 (ALERT)
- new net ADC_02_ALERT: U6.12 (ALERT)
Other:
- note added: "ADC-01"
- note added: "ADC_02"

Commit message: updated r values
Parts:
- R24, R25, R26, R27, R28, R29, R30, R31, R32, R33, R43, R44, R45, R46, R47, R48, R49, R50: value 20K -> 2K
Changed lines of the file:
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@@
 			)
 		)
-		(property "Value" "20K"
+		(property "Value" "2K"
 			(at 180.34 57.1499 0)
 			(effects
@@
 			)
 		)
-		(property "Value" "20K"
+		(property "Value" "2K"
 			(at 154.94 57.1499 0)
 			(effects
@@
 			)
 		)
-		(property "Value" "20K"
+		(property "Value" "2K"
 			(at 168.91 130.8099 0)
 			(effects
@@
 			)
 		)
-		(property "Value" "20K"
+		(property "Value" "2K"
 			(at 205.74 57.1499 0)
 			(effects
@@
 			)
 		)
-		(property "Value" "20K"
+		(property "Value" "2K"
 			(at 130.81 130.8099 0)
 			(effects
@@
 			)
 		)
-		(property "Value" "20K"
+		(property "Value" "2K"
 			(at 276.86 57.1499 0)
 			(effects
@@
 			)
 		)
-		(property "Value" "20K"
+		(property "Value" "2K"
 			(at 207.01 130.8099 0)
 			(effects
@@
 			)
 		)
-		(property "Value" "20K"
+		(property "Value" "2K"
 			(at 219.71 130.8099 0)
 			(effects
@@
 			)
 		)
-		(property "Value" "20K"
+		(property "Value" "2K"
 			(at 250.19 57.1499 0)
 			(effects
@@
 			)
 		)
-		(property "Value" "20K"
+		(property "Value" "2K"
 			(at 167.64 57.1499 0)
 			(effects
@@
 			)
 		)
-		(property "Value" "20K"
+		(property "Value" "2K"
 			(at 156.21 130.8099 0)
 			(effects
@@
 			)
 		)
-		(property "Value" "20K"
+		(property "Value" "2K"
 			(at 143.51 130.8099 0)
 			(effects
@@
 			)
 		)
-		(property "Value" "20K"
+		(property "Value" "2K"
 			(at 218.44 57.1499 0)
 			(effects
@@
 			)
 		)
-		(property "Value" "20K"
+		(property "Value" "2K"
 			(at 193.04 57.1499 0)
 			(effects
@@
 			)
 		)
-		(property "Value" "20K"
+		(property "Value" "2K"
 			(at 194.31 130.8099 0)
 			(effects
@@
 			)
 		)
-		(property "Value" "20K"
+		(property "Value" "2K"
 			(at 181.61 130.8099 0)
 			(effects
@@
 			)
 		)
-		(property "Value" "20K"
+		(property "Value" "2K"
 			(at 142.24 57.1499 0)
 			(effects
@@
 			)
 		)
-		(property "Value" "20K"
+		(property "Value" "2K"
 			(at 129.54 57.1499 0)
 			(effects
